File: Core.kicad_sch (KiCad schematic)
At the start: 5 parts, among them J11 Conn_01x05_Pin, J12 xcore, U5 M24C02-WMN

Commit message: wip
Parts:
- removed C17: 100nF, Capacitor_SMD:C_0402_1005Metric, symbol Device:C
- removed J11: Conn_01x05_Pin, Connector_PinHeader_2.54mm:PinHeader_1x05_P2.54mm_Vertical, symbol Connector:Conn_01x05_Pin
- removed J12: xcore, xcore:xcore, symbol xcore:xcore
- removed R15: 10k, Resistor_SMD:R_0402_1005Metric, symbol Device:R
- removed U5: M24C02-WMN, Package_SO:SOIC-8_3.9x4.9mm_P1.27mm, symbol Memory_EEPROM:M24C02-WMN
Other:
- note removed: "Identification for this Mainboard Version"
