File: Charger.kicad_sch (KiCad schematic)
At the start: 70 parts, among them J1 Screw_Terminal_01x02, J2 Conn_01x02, J21 Conn_01x06, J4 67800-8005, Q6 BSC0702LS, Q7 BSC0702LS, Q8 BSC0702LS, Q9 BSC0702LS, U2 LV2862XDDC, U27 BQ25756RRVR

Commit message: wip
Connections:
- no-connect marks 4 -> 8

Commit message: wip
Parts:
- added L2: 47uH, Inductor_SMD:L_Sunlord_SWPA5040S, symbol Device:L
- R4: value R -> 120k; footprint Resistor_SMD:R_0201_0603Metric -> Resistor_SMD:R_0603_1608Metric; JLC (none) -> C25808
- R81: value R -> 22k; footprint Resistor_SMD:R_0201_0603Metric -> Resistor_SMD:R_0603_1608Metric; JLC (none) -> C31850
Connections:
- net 5V: now also R4.1, L2.2; no longer R4.2, R81.1, U2.3 (FB)
- net at C7.1, D35.1 (K), U2.6 (SW): now also L2.1; no longer R4.1
- new net: R4.2, R81.1, U2.3 (FB)
Changed lines of the file:
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@@
 	)
 	(junction
+		(at 176.53 -27.94)
+		(diameter 0)
+		(color 0 0 0 0)
+	)
+	(junction
 		(at 109.22 55.88)
 		(diameter 0)
@@
 	)
 	(junction
+		(at 161.29 -35.56)
+		(diameter 0)
+		(color 0 0 0 0)
+	)
+	(junction
 		(at 422.91 124.46)
 		(diameter 0)
@@
 	)
 	(junction
-		(at 176.53 -27.94)
-		(diameter 0)
-		(color 0 0 0 0)
-	)
-	(junction
 		(at 82.55 55.88)
 		(diameter 0)
@@
 	(wire
 		(pts
-			(xy 161.29 -35.56) (xy 149.86 -35.56)
-		)
-		(stroke
-			(width 0)
-			(type default)
-		)
-	)
-	(wire
-		(pts
 			(xy 92.71 73.66) (xy 109.22 73.66)
 		)
@@
 	(wire
 		(pts
-			(xy 161.29 -27.94) (xy 176.53 -27.94)
+			(xy 151.13 102.87) (xy 185.42 102.87)
 		)
 		(stroke
@@
 	(wire
 		(pts
-			(xy 151.13 102.87) (xy 185.42 102.87)
+			(xy 176.53 -35.56) (xy 176.53 -27.94)
 		)
 		(stroke
@@
 	(wire
 		(pts
+			(xy 161.29 -35.56) (xy 176.53 -35.56)
+		)
+		(stroke
+			(width 0)
+			(type default)
+		)
+	)
+	(wire
+		(pts
 			(xy 109.22 73.66) (xy 109.22 55.88)
 		)
@@
 	(wire
 		(pts
+			(xy 149.86 -35.56) (xy 152.4 -35.56)
+		)
+		(stroke
+			(width 0)
+			(type default)
+		)
+	)
+	(wire
+		(pts
 			(xy 121.92 55.88) (xy 238.76 55.88)
 		)
@@
 	(wire
 		(pts
+			(xy 160.02 -35.56) (xy 161.29 -35.56)
+		)
+		(stroke
+			(width 0)
+			(type default)
+		)
+	)
+	(wire
+		(pts
 			(xy 294.64 129.54) (xy 289.56 129.54)
 		)
@@
 			)
 		)
-		(property "Value" "R"
+		(property "Value" "120k"
 			(at 163.83 -30.4801 0)
 			(effects
@@
 			)
 		)
-		(property "Footprint" "Resistor_SMD:R_0201_0603Metric"
+		(property "Footprint" "Resistor_SMD:R_0603_1608Metric"
 			(at 159.512 -31.75 90)
 			(effects
@@
 			)
 		)
+		(property "JLC" "C25808"
+			(at 161.29 -31.75 0)
+			(effects
+				(font
+					(size 1.27 1.27)
+				)
+				(hide yes)
+			)
+		)
 		(pin "1"
 		)
@@
 			)
 		)
-		(property "Value" "R"
+		(property "Value" "22k"
 			(at 163.83 -22.8601 0)
 			(effects
@@
 			)
 		)
-		(property "Footprint" "Resistor_SMD:R_0201_0603Metric"
+		(property "Footprint" "Resistor_SMD:R_0603_1608Metric"
 			(at 159.512 -24.13 90)
 			(effects
@@
 			)
 		)
+		(property "JLC" "C31850"
+			(at 161.29 -24.13 0)
+			(effects
+				(font
+					(size 1.27 1.27)
+				)
+				(hide yes)
+			)
+		)
 		(pin "1"
 		)
@@
 					(unit 1)
 				)
+			)
+		)
+	)
+	(symbol
+		(lib_id "Device:L")
+		(at 156.21 -35.56 90)
+		(unit 1)
+		(exclude_from_sim no)
+		(in_bom yes)
+		(on_board yes)
+		(dnp no)
+		(fields_autoplaced yes)
+		(property "Reference" "L2"
+			(at 156.21 -39.37 90)
+			(effects
+				(font
+					(size 1.27 1.27)
+				)
+			)
+		)
+		(property "Value" "47uH"
+			(at 156.21 -36.83 90)
+			(effects
+				(font
+					(size 1.27 1.27)
+				)
+			)
+		)
+		(property "Footprint" "Inductor_SMD:L_Sunlord_SWPA5040S"
+			(at 156.21 -35.56 0)
+			(effects
+				(font
+					(size 1.27 1.27)
+				)
+				(hide yes)
+			)
+		)
+		(property "Datasheet" "~"
+			(at 156.21 -35.56 0)
+			(effects
+				(font
+					(size 1.27 1.27)
+				)
+				(hide yes)
+			)
+		)
+		(property "Description" "Inductor"
+			(at 156.21 -35.56 0)
+			(effects
+				(font
+					(size 1.27 1.27)
+				)
+				(hide yes)
+			)
+		)
+		(property "JLC" "C86617"
+			(at 156.21 -35.56 90)
+			(effects
+				(font
+					(size 1.27 1.27)
+				)
+				(hide yes)
+			)
+		)
+		(pin "1"
+		)
+		(pin "2"
+		)
+		(instances
+			(project "hw-openmower-universal"
+				(path "/e12e8a63-1d1b-4736-9aba-a87a258b2b11/2930b75f-7142-4414-b99a-728851a6a7da/06123601-78a7-45a5-9135-d0172885f72e"
+					(reference "L2")
+					(unit 1)
+				)

Commit message: wip
Parts:
- removed J1: Screw_Terminal_01x02, TerminalBlock_Phoenix:TerminalBlock_Phoenix_MKDS-1,5-2-5.08_1x02_P5.08mm_Horizontal, symbol Connector:Screw_Terminal_01x02
- removed J2: Conn_01x02, Connector_AMASS:AMASS_XT30UPB-M_1x02_P5.0mm_Vertical, symbol Connector_Generic:Conn_01x02

Commit message: wip
Parts:
- removed C48, C76: 100nF@50V, Capacitor_SMD:C_0603_1608Metric, symbol Device:C
- removed J21: Conn_01x06, Connector_PinHeader_2.54mm:PinHeader_1x06_P2.54mm_Vertical, symbol Connector_Generic:Conn_01x06
- removed J4: 67800-8005, SATA-Molex-67800-8005:SATA-Molex-67800-8005, symbol SATA-Molex-67800-8005:67800-8005
- added C11: DNP, Capacitor_SMD:C_0603_1608Metric, symbol Device:C
- added C12: 100nF@50V, Capacitor_SMD:C_0603_1608Metric, symbol Device:C
- added C13, C16: 100nF@100V, Capacitor_SMD:C_0805_2012Metric, symbol Device:C
- added D16, D39: LED GREEN, LED_SMD:LED_0805_2012Metric, symbol Device:LED
- added J23: Conn_02x07_Odd_Even, Connector_PinHeader_2.54mm:PinHeader_2x07_P2.54mm_Vertical, symbol Connector_Generic:Conn_02x07_Odd_Even
- added R36, R79: 1k, Resistor_SMD:R_0805_2012Metric, symbol Device:R
- added R80: 220kR 0.1%, Resistor_SMD:R_0603_1608Metric, symbol Device:R
- added R86: 15k 0.1%, Resistor_SMD:R_0603_1608Metric, symbol Device:R
- added R87: 20k 0.1%, Resistor_SMD:R_0603_1608Metric, symbol Device:R
- added R88, R90, R92, R94, R95, R96: DNP, Resistor_SMD:R_0603_1608Metric, symbol Device:R
- added R89: 25.5k 0.5%, Resistor_SMD:R_0603_1608Metric, symbol Device:R
- added R91: 35.7k 1%, Resistor_SMD:R_0603_1608Metric, symbol Device:R
- added R93: 12.1k 1%, Resistor_SMD:R_0603_1608Metric, symbol Device:R
- R23: value 15k 0.1% -> 16.2k 0.1%; JLC C2692707 -> C22885
- R68, R69: footprint Resistor_SMD:R_0402_1005Metric -> Resistor_SMD:R_0603_1608Metric; JLC C25077 -> C22859
- R71: value 220kR 0.1% -> DNP; JLC C861231 -> (none); now not fitted
Connections:
- net 5V: now also D16.2 (A)
- net 5V_Main: now also D39.2 (A)
- net FB: now also C11.1, J23.1 (Pin_1), J23.11 (Pin_11), J23.13 (Pin_13), J23.3 (Pin_3), J23.5 (Pin_5), J23.7 (Pin_7), J23.9 (Pin_9); no longer R23.1, R71.1
- net FBG: now also C11.2, R80.2, R86.2, R87.2, R88.2, R89.2, R90.2, R91.2, R92.2, R93.2, R94.2, R95.2, R96.2
- net GND: now also C12.1, R36.2, R79.2
- net V_BATT_CHARGE: now also C12.2
- net at L4.2, Q8.1 (S), Q8.2 (S)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: now also C16.1
- net at D2.1 (K), U27.20 (BTST2): now also C16.2
- net at D26.1 (K), U27.26 (BTST1): now also C13.2
- net at L4.1, Q6.1 (S), Q6.2 (S)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: now also C13.1
- new net: J23.10 (Pin_10), R80.1, R86.1
- new net: D39.1 (K), R79.1
- new net: J23.8 (Pin_8), R23.1, R71.1
- new net: J23.12 (Pin_12), R93.1, R94.1
- new net: J23.14 (Pin_14), R95.1, R96.1
- new net: D16.1 (K), R36.1
- new net: J23.6 (Pin_6), R87.1, R88.1
- new net: J23.2 (Pin_2), R91.1, R92.1
- new net: J23.4 (Pin_4), R89.1, R90.1
- no-connect marks 8 -> 1
Other:
- note added: "3S RBot = 35.7 kOhms gives 4.08V cell end voltage."
- note added: "4S RBot = 25.5 kOhms gives 4.14V cell end voltage."
- note added: "5S RBot = 20.0 kOhms gives 4.14V cell end voltage."
- note added: "6S RBot = 16.2 kOhms gives 4.15V cell end voltage."
- note added: "7S RBot = 14.04 kOhms gives 4.12V cell end voltage. 14.04 = 220k and 15k in parallel"
- note added: "8S RBot = 12.1 kOhms gives 4.15V cell end voltage."
- note added: "Custom"
- note removed: "Connectors to join the PCBs when separated"
- note removed: "RBot = 14.04 kOhms gives 4.12V cell end voltage. 14.04 = 220k and 15k in parallel"
- moved on the sheet: R33

Commit message: wip
Parts:
- removed C114, C8: 22uF/25V, Capacitor_SMD:C_0805_2012Metric, symbol Device:C
- removed C2: 10uF@50V, Capacitor_SMD:C_1206_3216Metric, symbol Device:C
- removed C6, C7: 100nF@50V, Capacitor_SMD:C_0402_1005Metric, symbol Device:C
- removed D16: LED GREEN, LED_SMD:LED_0805_2012Metric, symbol Device:LED
- removed D34: SS14, Diode_SMD:D_SMA, symbol Diode:SS14
- removed D35: VS-2EFH02HM3/I, Diode_SMD:D_SMF, symbol Device:D_Schottky
- removed L2: 47uH, Inductor_SMD:L_Sunlord_SWPA5040S, symbol Device:L
- removed R2: 100k, Resistor_SMD:R_0402_1005Metric, symbol Device:R
- removed R36: 1k, Resistor_SMD:R_0805_2012Metric, symbol Device:R
- removed R4: 120k, Resistor_SMD:R_0603_1608Metric, symbol Device:R
- removed R81: 22k, Resistor_SMD:R_0603_1608Metric, symbol Device:R
- removed U2: LV2862XDDC, Package_TO_SOT_SMD:SOT-23-6, symbol Regulator_Switching:LV2862XDDC
Connections:
- net 5V_Main is gone; now on net 5V: D39.2 (A)
Other:
- note removed: "Diode can be removed, when DCDC is not in the design"
- note removed: "Generates 5V on the sub-PCB. This is only necessary when splitting the PCB and using it in stand-alone operation. If you design an integrated solution, use the 5V from the main DCDC instead to save on cost and solution size."
- moved on the sheet: D39, R79

Commit message: wip
Parts:
- removed J23: Conn_02x07_Odd_Even, Connector_PinHeader_2.54mm:PinHeader_2x07_P2.54mm_Vertical, symbol Connector_Generic:Conn_02x07_Odd_Even
- removed R89: 25.5k 0.5%, Resistor_SMD:R_0603_1608Metric, symbol Device:R
- removed R90, R92: DNP, Resistor_SMD:R_0603_1608Metric, symbol Device:R
- removed R91: 35.7k 1%, Resistor_SMD:R_0603_1608Metric, symbol Device:R
- added J2: Conn_02x04_Odd_Even, Connector_PinHeader_2.54mm:PinHeader_2x04_P2.54mm_Vertical, symbol Connector_Generic:Conn_02x04_Odd_Even
- added JP3: SolderJumper_2_Open, Jumper:SolderJumper-2_P1.3mm_Open_Pad1.0x1.5mm, symbol Jumper:SolderJumper_2_Open
Connections:
- net FB: now also J2.1 (Pin_1), J2.3 (Pin_3), J2.5 (Pin_5), J2.7 (Pin_7), JP3.2 (B)
- net at R80.1, R86.1: now also J2.6 (Pin_6)
- net at R23.1, R71.1: now also J2.4 (Pin_4)
- net at R93.1, R94.1: now also J2.8 (Pin_8)
- net at R95.1, R96.1: now also JP3.1 (A)
- net at R87.1, R88.1: now also J2.2 (Pin_2)
Other:
- note removed: "3S RBot = 35.7 kOhms gives 4.08V cell end voltage."
- note removed: "4S RBot = 25.5 kOhms gives 4.14V cell end voltage."

Commit message: wip
Parts:
- removed R20: 47kR, Resistor_SMD:R_0603_1608Metric, symbol Device:R
- added J4: Conn_02x05_Odd_Even, Connector_PinHeader_2.54mm:PinHeader_2x05_P2.54mm_Vertical, symbol Connector_Generic:Conn_02x05_Odd_Even
- added JP4: SolderJumper_2_Bridged, Jumper:SolderJumper-2_P1.3mm_Bridged_Pad1.0x1.5mm, symbol Jumper:SolderJumper_2_Bridged
- added R2: 47kR, Resistor_SMD:R_0603_1608Metric, symbol Device:R
- added R36: 16.2k 0.1%, Resistor_SMD:R_0603_1608Metric, symbol Device:R
- added R4: 25k 0.1%, Resistor_SMD:R_0603_1608Metric, symbol Device:R
- added R81: 12.1k 1%, Resistor_SMD:R_0603_1608Metric, symbol Device:R
- added R89: 10k, Resistor_SMD:R_0603_1608Metric, symbol Device:R
- J2: JLC (none) -> C5383105
Connections:
- net GND: now also R2.1, R36.2, R4.2, R81.2, R89.2
- net ICHG: now reaches U27.9 (ICHG)
- net ICHG: now also JP4.2 (B)
- new net: J4.1 (Pin_1), J4.3 (Pin_3), J4.5 (Pin_5), J4.7 (Pin_7), J4.9 (Pin_9), JP4.1 (A)
- new net: J4.10 (Pin_10), R2.2
- new net: J4.2 (Pin_2), R89.1
- new net: J4.4 (Pin_4), R81.1
- new net: J4.6 (Pin_6), R36.1
- new net: J4.8 (Pin_8), R4.1

Commit message: First Version worth testing
Parts:
- C83: value 470nF@25V -> 470nF/25V
- R23, R36: value 16.2k 0.1% -> 16.2k 1%
Changed lines of the file:
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@@
 			)
 		)
-		(property "Value" "470nF@25V"
+		(property "Value" "470nF/25V"
 			(at 386.08 151.13 90)
 			(effects
@@
 			)
 		)
-		(property "Value" "16.2k 0.1%"
+		(property "Value" "16.2k 1%"
 			(at 118.11 226.0599 0)
 			(effects
@@
 			)
 		)
-		(property "Value" "16.2k 0.1%"
+		(property "Value" "16.2k 1%"
 			(at 294.64 215.8999 0)
 			(effects
