File: subpcb_logic.kicad_sch (KiCad schematic)
At the start: 56 parts, among them J13 Screw_Terminal_01x02, J14 Conn_01x02, J15 Conn_01x04, J16 67800-8005, J18 67800-8005, J23 Conn_01x02, J24 Conn_01x02, J25 67800-8005, J26 67800-8005, J27 67800-8005, J28 Conn_01x03_Male, J29 Conn_01x03_Male, J30 Conn_01x03_Male, J31 Conn_01x03_Pin, J32 Conn_02x08_Odd_Even, J51 Conn_01x03_Male, J52 Conn_01x03_Male, J53 Conn_01x03_Male, J54 Conn_01x03_Male, J55 Conn_01x03_Male, M1 Fan, Q1 BSS138, Q2 BSS138, U6 AS-RTK2B-MICRO-F9P-L1L2SMATH-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, U7 TXS0108EPW

Commit message: wip
Parts:
- removed J23: Conn_01x02, Connector_JST:JST_XH_B2B-XH-A_1x02_P2.50mm_Vertical, symbol Connector_Generic:Conn_01x02
- removed J29, J51, J53, J55: Conn_01x03_Male, Connector_JST:JST_XH_B3B-XH-A_1x03_P2.50mm_Vertical, symbol Connector:Conn_01x03_Male
- removed J32: Conn_02x08_Odd_Even, Connector_PinHeader_2.54mm:PinHeader_2x08_P2.54mm_Vertical, symbol Connector_Generic:Conn_02x08_Odd_Even
- added C17: 100nF, Capacitor_SMD:C_0402_1005Metric, symbol Device:C
- added C34: 220uF@80V, Capacitor_THT:CP_Radial_D10.0mm_P5.00mm, symbol Device:C_Polarized
- added J11: Conn_01x05_Pin, Connector_PinHeader_2.54mm:PinHeader_1x05_P2.54mm_Vertical, symbol Connector:Conn_01x05_Pin
- added J12: xcore, xcore:xcore, symbol xcore:xcore
- added R15: 10k, Resistor_SMD:R_0402_1005Metric, symbol Device:R
- added U5: M24C02-WMN, Package_SO:SOIC-8_3.9x4.9mm_P1.27mm, symbol Memory_EEPROM:M24C02-WMN
- J28, J30, J52, J54: footprint Connector_JST:JST_XH_B3B-XH-A_1x03_P2.50mm_Vertical -> Connector_PinHeader_2.54mm:PinHeader_1x03_P2.54mm_Vertical
Connections:
- net 3.3V: now also J12.19 (3.3V_Output), J12.21 (3.3V_Output)
- net 5V: now also J12.1 (5V_Input), J12.11 (5V_Input), J12.13 (5V_Input), J12.15 (5V_Input), J12.17 (5V_Input), J12.3 (5V_Input), J12.5 (5V_Input), J12.7 (5V_Input), J12.9 (5V_Input)
- net AGPIO0: now also J12.149 (AGPIO0)
- net AGPIO1: now also J12.151 (AGPIO1)
- net AGPIO2: now also J12.153 (AGPIO2)
- net AGPIO3: now also J12.155 (AGPIO3)
- net AGPIO4: now also J12.157 (AGPIO4)
- net AGPIO5: now also J12.159 (AGPIO5)
- net GND: now also C17.2, C34.2, J11.5 (Pin_5), J12.10 (GND), J12.104 (GND), J12.114 (GND), J12.12 (GND), J12.120 (GND), J12.14 (GND), J12.147 (GND), J12.16 (GND), J12.168 (GND), J12.173 (GND), J12.174 (GND), J12.179 (GND), J12.18 (GND), J12.180 (GND), J12.185 (GND), J12.186 (GND), J12.191 (GND), J12.192 (GND), J12.197 (GND), J12.198 (GND), J12.2 (GND), J12.203 (GND), J12.204 (GND), J12.23 (GND), J12.24 (GND), J12.29 (GND), J12.30 (GND), J12.35 (GND), J12.36 (GND), J12.39 (GND), J12.4 (GND), J12.40 (GND), J12.45 (GND), J12.46 (GND), J12.51 (GND), J12.52 (GND), J12.55 (GND), J12.56 (GND), J12.6 (GND), J12.61 (GND), J12.62 (GND), J12.67 (GND), J12.68 (GND), J12.71 (GND), J12.72 (GND), J12.73 (GND), J12.74 (GND), J12.8 (GND), J12.82 (GND), J12.87 (GND), J12.90 (GND), J12.SH1 (GND), J12.SH2 (GND), U5.1 (E0), U5.2 (E1), U5.3 (E2), U5.4 (VSS)
- net GPIO1: now also J12.131 (GPIO1)
- net GPIO10: now also J12.148 (GPIO10)
- net GPIO11: now also J12.146 (GPIO11)
- net GPIO12: now also J12.144 (GPIO12)
- net GPIO13: now also J12.142 (GPIO13)
- net GPIO14: now also J12.140 (GPIO14)
- net RASPI_FAN_ON: now also J12.164 (CM_FAN_PWM)
- net STM_SWCLK: now also J12.160 (SWCLK)
- net STM_SWDIO: now also J12.162 (SWDIO)
- net UART1.RX: now also J12.81 (UART1.RX)
- net UART1.TX: now also J12.79 (UART1.TX)
- net UART10.RX: now also J12.103 (UART10.RX)
- net UART10.TX: now also J12.101 (UART10.TX)
- net UART2.RX: now also J12.91 (UART2.RX)
- net UART2.TX: now also J12.89 (UART2.TX)
- net UART4.RX: now also J12.85 (UART4.RX)
- net UART4.TX: now also J12.83 (UART4.TX)
- net UART6.RX: now also J12.77 (UART6.RX)
- net UART6.TX: now also J12.75 (UART6.TX)
- net UART7.RX: now also J12.95 (UART7.RX)
- net UART7.TX: now also J12.93 (UART7.TX)
- net UART8.RX: now also J12.99 (UART8.RX)
- net UART8.TX: now also J12.97 (UART8.TX)
- net V_BATTERY: now also C34.1
- new net 3.3V_Out: C17.1, J11.1 (Pin_1), R15.1, U5.8 (VCC)
- new net ETH1.LED_G: J12.54 (ETH1.LED_Green)
- new net ETH1.LED_Y: J12.53 (ETH1.LED_Yellow)
- new net ETH1.PAIR_A_N: J12.47 (ETH1.Pair_A-)
- new net ETH1.PAIR_A_P: J12.49 (ETH1.Pair_A+)
- new net ETH1.PAIR_B_N: J12.48 (ETH1.Pair_B-)
- new net ETH1.PAIR_B_P: J12.50 (ETH1.Pair_B+)
- new net ETH1.PAIR_C_N: J12.41 (ETH1.Pair_C-)
- new net ETH1.PAIR_C_P: J12.43 (ETH1.Pair_C+)
- new net ETH1.PAIR_D_N: J12.42 (ETH1.Pair_D-)
- new net ETH1.PAIR_D_P: J12.44 (ETH1.Pair_D+)
- new net ETH2.LED_G: J12.38 (ETH2.LED_Green)
- new net ETH2.LED_Y: J12.37 (ETH2.LED_Yellow)
- new net ETH2.PAIR_A_N: J12.31 (ETH2.Pair_A-)
- new net ETH2.PAIR_A_P: J12.33 (ETH2.Pair_A+)
- new net ETH2.PAIR_B_N: J12.32 (ETH2.Pair_B-)
- new net ETH2.PAIR_B_P: J12.34 (ETH2.Pair_B+)
- new net ETH2.PAIR_C_N: J12.25 (ETH2.Pair_C-)
- new net ETH2.PAIR_C_P: J12.27 (ETH2.Pair_C+)
- new net ETH2.PAIR_D_N: J12.26 (ETH2.Pair_D-)
- new net ETH2.PAIR_D_P: J12.28 (ETH2.Pair_D+)
- new net I2C4_ID.SCL: J11.3 (Pin_3), J12.102 (ID_I2C.SCL), U5.6 (SCL)
- new net I2C4_ID.SDA: J11.2 (Pin_2), J12.100 (ID_I2C.SDA), U5.5 (SDA)
- new net USBH1.N: J12.177 (USB0_D-)
- new net USBH1.P: J12.175 (USB0_D+)
- new net USBH2.N: J12.183 (USB1_D-)
- new net USBH2.P: J12.181 (USB1_D+)
- new net ~{WC}: J11.4 (Pin_4), R15.2, U5.7 (~{WC})
- no-connect marks 25 -> 71
Other:
- removed sheet Amplifier
- removed sheet Core
- note added: "Identification for this Mainboard Version"
- note removed: "Optional: Expansion Port"

Commit message: wip
Parts:
- removed R17, R64, R87, R88, R89: 150R, Resistor_SMD:R_0603_1608Metric, symbol Device:R
- added R1, R3, R5, R6, R83, R84, R85: 150R, Resistor_SMD:R_0603_1608Metric, symbol Device:R
Connections:
- net AGPIO1: now also J16.4, R18.1; no longer J12.151 (AGPIO1)
- net AGPIO2: now also J25.4, R39.1; no longer J12.153 (AGPIO2)
- net AGPIO3: now also J27.4, R40.1; no longer J12.155 (AGPIO3)
- net AGPIO4: now also J18.4, R42.1; no longer J12.157 (AGPIO4), R63.2
- net AGPIO5: now also J26.4, R63.1; no longer J12.159 (AGPIO5)
- net GPIO10: now also R41.2, U7.6 (A5); no longer R19.2, U7.9 (A8)
- net GPIO11: now also R38.2, U7.7 (A6); no longer R37.2, U7.8 (A7)
- net GPIO12: now also R37.2, U7.8 (A7); no longer R38.2, U7.7 (A6)
- net GPIO13: now also R19.2, U7.9 (A8); no longer R41.2, U7.6 (A5)
- net UART1.TX: now also J16.3, R1.1; no longer J12.79 (UART1.TX)
- net UART10.TX: now also J18.3, R85.1; no longer J12.101 (UART10.TX), R18.1
- net UART2.TX: now also J25.3, R3.1; no longer J12.89 (UART2.TX), R39.1
- net UART4.TX: now also J27.3, R5.1; no longer J12.83 (UART4.TX), R42.1
- net UART6.TX: now also J26.3, R6.1; no longer J12.75 (UART6.TX), R40.1
- net UART7.TX: now also R83.1; no longer J12.93 (UART7.TX)
- net UART8.TX: now also R84.1; no longer J12.97 (UART8.TX)
- net at R39.2: now also J12.153 (AGPIO2); no longer J25.3
- net at R18.2: now also J12.151 (AGPIO1); no longer J18.3
- net at R40.2: now also J12.155 (AGPIO3); no longer J26.3
- net at R42.2: now also J12.157 (AGPIO4); no longer J27.3
- new net: J12.83 (UART4.TX), R5.2
- new net: J12.97 (UART8.TX), R84.2
- new net: J12.79 (UART1.TX), R1.2
- new net: J12.159 (AGPIO5), R63.2
- new net: J12.89 (UART2.TX), R3.2
- new net: J12.101 (UART10.TX), R85.2
- new net: J12.75 (UART6.TX), R6.2
- new net: J12.93 (UART7.TX), R83.2

Commit message: wip
Parts:
- removed J11: Conn_01x05_Pin, Connector_PinHeader_2.54mm:PinHeader_1x05_P2.54mm_Vertical, symbol Connector:Conn_01x05_Pin
- added TP2: TestPoint_2Pole, Connector_PinHeader_1.00mm:PinHeader_1x02_P1.00mm_Vertical, symbol Connector:TestPoint_2Pole
Connections:
- net GND: now also TP2.2
- net I2C1.SCL: now also J12.94 (I2C1.SCL)
- net I2C1.SDA: now also J12.92 (I2C1.SDA)
- net ~{WC}: now also TP2.1
- no-connect marks 71 -> 69

Commit message: wip
Parts:
- added C2, C48, C6, C7, C8: 22pF/50V, Capacitor_SMD:C_0603_1608Metric, symbol Device:C
- added J1: Conn_01x04, Connector_JST:JST_XH_B4B-XH-A_1x04_P2.50mm_Vertical, symbol Connector_Generic:Conn_01x04
Connections:
- net 5V: now also J1.1 (Pin_1)
- net AGPIO1: now also C48.1
- net AGPIO2: now also C8.1
- net AGPIO3: now also C7.1
- net AGPIO4: now also C2.1
- net AGPIO5: now also C6.1
- net GND: now also C2.2, C48.2, C6.2, C7.2, C8.2, J1.4 (Pin_4)
- net UART10.RX: now also J1.3 (Pin_3)
- net UART10.TX: now also J1.2 (Pin_2)

Commit message: wip
Parts:
- TP2: footprint Connector_PinHeader_1.00mm:PinHeader_1x02_P1.00mm_Vertical -> Connector_PinHeader_2.54mm:PinHeader_1x02_P2.54mm_Vertical
Changed lines of the file:
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@@
 			)
 		)
-		(property "Footprint" "Connector_PinHeader_1.00mm:PinHeader_1x02_P1.00mm_Vertical"
+		(property "Footprint" "Connector_PinHeader_2.54mm:PinHeader_1x02_P2.54mm_Vertical"
 			(at 71.12 551.18 0)
 			(effects

Commit message: wip
Parts:
- removed TP2: TestPoint_2Pole, Connector_PinHeader_2.54mm:PinHeader_1x02_P2.54mm_Vertical, symbol Connector:TestPoint_2Pole
- added TP2: TestPoint, Connector_Pin:Pin_D1.4mm_L8.5mm_W2.8mm_FlatFork, symbol Connector:TestPoint
Connections:
- net 5V: now also J28.3 (Pin_3), J30.3 (Pin_3), J52.3 (Pin_3), J54.3 (Pin_3); no longer J28.1 (Pin_1), J30.1 (Pin_1), J52.1 (Pin_1), J54.1 (Pin_1)
- net GND: now also J28.1 (Pin_1), J30.1 (Pin_1), J52.1 (Pin_1), J54.1 (Pin_1); no longer J28.3 (Pin_3), J30.3 (Pin_3), J52.3 (Pin_3), J54.3 (Pin_3)
- net ~{WC}: now also TP2.1
Other:
- moved on the sheet: J28, J30, J52, J54
Changed lines of the file:
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@@
 	(symbol
 		(lib_id "Connector:Conn_01x03_Male")
-		(at 373.38 214.63 180)
+		(at 373.38 214.63 0)
+		(mirror y)
 		(unit 1)
 		(exclude_from_sim no)
@@
 		(dnp no)
 		(property "Reference" "J52"
-			(at 374.0912 212.9028 0)
+			(at 374.0912 216.3572 0)
 			(effects
 				(font
@@
 		)
 		(property "Value" "Conn_01x03_Male"
-			(at 374.0912 215.2142 0)
+			(at 374.0912 214.0458 0)
 			(effects
 				(font
@@
 	)
 	(symbol
-		(lib_id "Connector:TestPoint_2Pole")
-		(at 71.12 551.18 0)
-		(unit 1)
-		(exclude_from_sim no)
-		(in_bom yes)
-		(on_board yes)
-		(dnp no)
-		(fields_autoplaced yes)
-		(property "Reference" "TP2"
-			(at 71.12 546.1 0)
-			(effects
-				(font
-					(size 1.27 1.27)
-				)
-			)
-		)
-		(property "Value" "TestPoint_2Pole"
-			(at 71.12 548.64 0)
-			(effects
-				(font
-					(size 1.27 1.27)
-				)
-			)
-		)
-		(property "Footprint" "Connector_PinHeader_2.54mm:PinHeader_1x02_P2.54mm_Vertical"
-			(at 71.12 551.18 0)
-			(effects
-				(font
-					(size 1.27 1.27)
-				)
-				(hide yes)
-			)
-		)
-		(property "Datasheet" "~"
-			(at 71.12 551.18 0)
-			(effects
-				(font
-					(size 1.27 1.27)
-				)
-				(hide yes)
-			)
-		)
-		(property "Description" "2-polar test point"
-			(at 71.12 551.18 0)
-			(effects
-				(font
-					(size 1.27 1.27)
-				)
-				(hide yes)
-			)
-		)
-		(pin "1"
-		)
-		(pin "2"
-		)
-		(instances
-			(project "hw-openmower-universal"
-				(path "/e12e8a63-1d1b-4736-9aba-a87a258b2b11/becd8bd3-4d11-46de-85b5-377ba260c0f8"
-					(reference "TP2")
-					(unit 1)
-				)
-			)
-		)
-	)
-	(symbol
 		(lib_id "Device:R")
 		(at 172.72 461.01 90)
@@
 	(symbol
 		(lib_id "Connector:Conn_01x03_Male")
-		(at 373.38 232.41 180)
+		(at 373.38 232.41 0)
+		(mirror y)
 		(unit 1)
 		(exclude_from_sim no)
@@
 		(dnp no)
 		(property "Reference" "J54"
-			(at 374.0912 230.6828 0)
+			(at 374.0912 234.1372 0)
 			(effects
 				(font
@@
 		)
 		(property "Value" "Conn_01x03_Male"
-			(at 374.0912 232.9942 0)
+			(at 374.0912 231.8258 0)
 			(effects
 				(font
@@
 	)
 	(symbol
-		(lib_id "power:GND")
-		(at 76.2 551.18 0)
-		(mirror y)
-		(unit 1)
-		(exclude_from_sim no)
-		(in_bom yes)
-		(on_board yes)
-		(dnp no)
-		(property "Reference" "#PWR02"
-			(at 76.2 557.53 0)
-			(effects
-				(font
-					(size 1.27 1.27)
-				)
-				(hide yes)
-			)
-		)
-		(property "Value" "GND"
-			(at 76.2001 554.99 90)
-			(effects
-				(font
-					(size 1.27 1.27)
-				)
-				(justify right)
-			)
-		)
-		(property "Footprint" ""
-			(at 76.2 551.18 0)
-			(effects
-				(font
-					(size 1.27 1.27)
-				)
-				(hide yes)
-			)
-		)
-		(property "Datasheet" ""
-			(at 76.2 551.18 0)
-			(effects
-				(font
-					(size 1.27 1.27)
-				)
-				(hide yes)
-			)
-		)
-		(property "Description" "Power symbol creates a global label with name \"GND\" , ground"
-			(at 76.2 551.18 0)
-			(effects
-				(font
-					(size 1.27 1.27)
-				)
-				(hide yes)
-			)
-		)
-		(pin "1"
-		)
-		(instances
-			(project "hw-openmower-universal"
-				(path "/e12e8a63-1d1b-4736-9aba-a87a258b2b11/becd8bd3-4d11-46de-85b5-377ba260c0f8"
-					(reference "#PWR02")
-					(unit 1)
-				)
-			)
-		)
-	)
-	(symbol
 		(lib_id "Device:R")
 		(at 133.35 172.72 90)
@@
 	(symbol
 		(lib_id "Connector:Conn_01x03_Male")
-		(at 373.38 196.85 180)
+		(at 373.38 196.85 0)
+		(mirror y)
 		(unit 1)
 		(exclude_from_sim no)
@@
 		(dnp no)
 		(property "Reference" "J30"
-			(at 374.0912 195.1228 0)
+			(at 374.0912 198.5772 0)
 			(effects
 				(font
@@
 		)
 		(property "Value" "Conn_01x03_Male"
-			(at 374.0912 197.4342 0)
+			(at 374.0912 196.2658 0)
 			(effects
 				(font
@@
 	)
 	(symbol
+		(lib_id "Connector:TestPoint")
+		(at 66.04 551.18 0)
+		(unit 1)
+		(exclude_from_sim no)
+		(in_bom yes)
+		(on_board yes)
+		(dnp no)
+		(fields_autoplaced yes)
+		(property "Reference" "TP2"
+			(at 68.58 546.6079 0)
+			(effects
+				(font
+					(size 1.27 1.27)
+				)
+				(justify left)
+			)
+		)
+		(property "Value" "TestPoint"
+			(at 68.58 549.1479 0)
+			(effects
+				(font
+					(size 1.27 1.27)
+				)
+				(justify left)
+			)
+		)
+		(property "Footprint" "Connector_Pin:Pin_D1.4mm_L8.5mm_W2.8mm_FlatFork"
+			(at 71.12 551.18 0)
+			(effects
+				(font
+					(size 1.27 1.27)
+				)
+				(hide yes)
+			)
+		)
+		(property "Datasheet" "~"
+			(at 71.12 551.18 0)
+			(effects
+				(font
+					(size 1.27 1.27)
+				)
+				(hide yes)
+			)
+		)
+		(property "Description" "test point"
+			(at 66.04 551.18 0)
+			(effects
+				(font
+					(size 1.27 1.27)
+				)
+				(hide yes)
+			)
+		)
+		(pin "1"
+		)
+		(instances
+			(project "hw-openmower-universal"
+				(path "/e12e8a63-1d1b-4736-9aba-a87a258b2b11/becd8bd3-4d11-46de-85b5-377ba260c0f8"
+					(reference "TP2")
+					(unit 1)
+				)
+			)
+		)
+	)
+	(symbol
 		(lib_id "Device:R")
 		(at 71.12 424.18 90)
@@
 	(symbol
 		(lib_id "Connector:Conn_01x03_Male")
-		(at 373.38 179.07 180)
+		(at 373.38 179.07 0)
+		(mirror y)
 		(unit 1)
 		(exclude_from_sim no)
@@
 		(dnp no)
 		(property "Reference" "J28"
-			(at 374.0912 177.3428 0)
+			(at 374.0912 180.7972 0)
 			(effects
 				(font
@@
 		)
 		(property "Value" "Conn_01x03_Male"
-			(at 374.0912 179.6542 0)
+			(at 374.0912 178.4858 0)
 			(effects
 				(font

Commit message: wip
Parts:
- J13: JLC (none) -> C557665
- J14: JLC (none) -> C428721
- J16, J18, J25, J26, J27: JLC (none) -> C7500843
- J31, U6: now not fitted

Commit message: First Version worth testing
Parts:
- Q1, Q2: value BSS138 -> AO3400A; JLC C3040446 -> C20917
- R25, R53: value 150 -> 150R
Connections:
- net GPIO14: no longer names the net of J12.140 (GPIO14)
- no-connect marks 69 -> 70
Changed lines of the file:
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@@
 	)
 	(no_connect
+		(at 181.61 417.83)
+	)
+	(no_connect
 		(at 181.61 397.51)
 	)
@@
 		)
 	)
-	(wire
-		(pts
-			(xy 181.61 417.83) (xy 170.18 417.83)
-		)
-		(stroke
-			(width 0)
-			(type default)
-		)
-	)
 	(bus
 		(pts
@@
 		)
 	)
-	(label "GPIO14"
-		(at 170.18 417.83 0)
-		(fields_autoplaced yes)
-		(effects
-			(font
-				(size 1.27 1.27)
-			)
-			(justify left bottom)
-		)
-	)
 	(label "5V"
 		(at 218.44 46.99 90)
@@
 			)
 		)
-		(property "Value" "150"
+		(property "Value" "150R"
 			(at 497.84 204.47 90)
 			(effects
@@
 			)
 		)
-		(property "LCSC" ""
-			(at 497.84 208.28 0)
-			(effects
-				(font
-					(size 1.27 1.27)
-				)
-				(hide yes)
-			)
-		)
 		(property "JLC" "C17471"
 			(at 497.84 208.28 0)
@@
 			)
 		)
-		(property "LCSC" ""
-			(at 373.38 214.63 0)
-			(effects
-				(font
-					(size 1.27 1.27)
-				)
-				(hide yes)
-			)
-		)
 		(property "JLC" "C144394"
 			(at 373.38 214.63 0)
@@
 			)
 		)
-		(property "Value" "150"
+		(property "Value" "150R"
 			(at 447.04 120.65 90)
 			(effects
@@
 			)
 		)
-		(property "LCSC" ""
-			(at 447.04 124.46 0)
-			(effects
-				(font
-					(size 1.27 1.27)
-				)
-				(hide yes)
-			)
-		)
 		(property "JLC" "C17471"
 			(at 447.04 124.46 0)
@@
 			)
 		)
-		(property "LCSC" ""
-			(at 72.39 256.54 0)
-			(effects
-				(font
-					(size 1.27 1.27)
-				)
-				(hide yes)
-			)
-		)
 		(property "JLC" "C144395"
 			(at 72.39 256.54 0)
@@
 			)
 		)
-		(property "LCSC" ""
-			(at 490.22 215.9 0)
-			(effects
-				(font
-					(size 1.27 1.27)
-				)
-				(hide yes)
-			)
-		)
 		(property "JLC" "C17414"
 			(at 490.22 215.9 0)
@@
 			)
 		)
-		(property "LCSC" ""
-			(at 373.38 232.41 0)
-			(effects
-				(font
-					(size 1.27 1.27)
-				)
-				(hide yes)
-			)
-		)
 		(property "JLC" "C144394"
 			(at 373.38 232.41 0)
@@
 			)
 		)
-		(property "Value" "BSS138"
+		(property "Value" "AO3400A"
 			(at 466.09 125.7299 0)
 			(effects
@@
 			)
 		)
-		(property "LCSC" ""
-			(at 459.74 124.46 0)
-			(effects
-				(font
-					(size 1.27 1.27)
-				)
-				(hide yes)
-			)
-		)
 		(property "Part Number" "AP2300"
 			(at 459.74 124.46 0)
@@
 			)
 		)
-		(property "JLC" "C3040446"
+		(property "JLC" "C20917"
 			(at 459.74 124.46 0)
 			(effects
@@
 			)
 		)
-		(property "LCSC" ""
-			(at 504.19 194.31 0)
-			(effects
-				(font
-					(size 1.27 1.27)
-				)
-				(hide yes)
-			)
-		)
 		(property "Part Number" "AS160-M"
 			(at 504.19 194.31 0)
@@
 			)
 		)
-		(property "LCSC" ""
-			(at 162.56 256.54 0)
-			(effects
-				(font
-					(size 1.27 1.27)
-				)
-				(hide yes)
-			)
-		)
 		(property "JLC" "C144395"
 			(at 162.56 256.54 0)
@@
 			)
 		)
-		(property "LCSC" ""
-			(at 175.26 172.72 0)
-			(effects
-				(font
-					(size 1.27 1.27)
-				)
-				(hide yes)
-			)
-		)
 		(property "JLC" "C2910525"
 			(at 175.26 172.72 0)
@@
 			)
 		)
-		(property "LCSC" ""
-			(at 373.38 196.85 0)
-			(effects
-				(font
-					(size 1.27 1.27)
-				)
-				(hide yes)
-			)
-		)
 		(property "JLC" "C144394"
 			(at 373.38 196.85 0)
@@
 			)
 		)
-		(property "Value" "BSS138"
+		(property "Value" "AO3400A"
 			(at 516.89 209.5499 0)
 			(effects
@@
 			)
 		)
-		(property "LCSC" ""
-			(at 510.54 208.28 0)
-			(effects
-				(font
-					(size 1.27 1.27)
-				)
-				(hide yes)
-			)
-		)
 		(property "Part Number" "AP2300"
 			(at 510.54 208.28 0)
@@
 			)
 		)
-		(property "JLC" "C3040446"
+		(property "JLC" "C20917"
 			(at 510.54 208.28 0)
 			(effects
@@
 			)
 		)
-		(property "LCSC" ""
-			(at 439.42 132.08 0)
-			(effects
-				(font
-					(size 1.27 1.27)
-				)
-				(hide yes)
-			)
-		)
 		(property "JLC" "C17414"
 			(at 439.42 132.08 0)
@@
 			)
 		)
-		(property "LCSC" ""
-			(at 513.08 195.58 0)
-			(effects
-				(font
-					(size 1.27 1.27)
-				)
-				(hide yes)
-			)
-		)
 		(property "Part Number" "DZ254R-11-02-63"
 			(at 513.08 195.58 0)
@@
 			(at 373.38 179.07 0)
 			(effects
-				(font
-					(size 1.27 1.27)
-				)
-				(hide yes)
-			)
-		)
-		(property "LCSC" ""
-			(at 373.38 179.07 0)
-			(effects
