File: xESC.kicad_sch (KiCad schematic)
At the start: 43 parts, among them J22 Screw_Terminal_01x03, J36 Conn_02x03_Odd_Even, J39 Screw_Terminal_01x02, J42 Conn_01x02, J45 67800-8005, J48 Conn_01x05, U10 xESC2, U20 2.54mm 2x2 socket, U23 2.54mm 2x2 socket, U26 2.54mm 2x2 socket, U28 LV2862XDDC, U32 2.54mm 1x6 socket, U35 2.54mm 1x6 socket, U38 2.54mm 1x9 socket, U41 2.54mm 1x5 socket

Commit message: wip
Parts:
- removed R78: 150R, Resistor_SMD:R_0603_1608Metric, symbol Device:R
Connections:
- net TX: now also J45.2, J48.4 (Pin_4); no longer U10.12 (MOSI/TX)
- net at R43.2: now also U10.12 (MOSI/TX); no longer J45.2
Other:
- moved on the sheet: R43
Changed lines of the file:
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@@
 	(wire
 		(pts
-			(xy 100.33 139.7) (xy 142.24 139.7)
-		)
-		(stroke
-			(width 0)
-			(type default)
-		)
-	)
-	(wire
-		(pts
 			(xy 185.42 102.87) (xy 203.2 102.87)
 		)
@@
 	(wire
 		(pts
-			(xy 318.77 46.99) (xy 323.85 46.99)
-		)
-		(stroke
-			(width 0)
-			(type default)
-		)
-	)
-	(wire
-		(pts
 			(xy 156.21 46.99) (xy 171.45 46.99)
 		)
@@
 	(wire
 		(pts
+			(xy 134.62 139.7) (xy 142.24 139.7)
+		)
+		(stroke
+			(width 0)
+			(type default)
+		)
+	)
+	(wire
+		(pts
 			(xy 214.63 99.06) (xy 214.63 113.03)
 		)
@@
 	(wire
 		(pts
+			(xy 283.21 17.78) (xy 283.21 33.02)
+		)
+		(stroke
+			(width 0)
+			(type default)
+		)
+	)
+	(wire
+		(pts
 			(xy 82.55 36.83) (xy 96.52 36.83)
 		)
@@
 	(wire
 		(pts
+			(xy 100.33 139.7) (xy 127 139.7)
+		)
+		(stroke
+			(width 0)
+			(type default)
+		)
+	)
+	(wire
+		(pts
 			(xy 124.46 100.33) (xy 142.24 100.33)
 		)
@@
 	(wire
 		(pts
-			(xy 304.8 46.99) (xy 311.15 46.99)
+			(xy 304.8 46.99) (xy 323.85 46.99)
 		)
 		(stroke
@@
 	(wire
 		(pts
-			(xy 283.21 17.78) (xy 283.21 22.86)
-		)
-		(stroke
-			(width 0)
-			(type default)
-		)
-	)
-	(wire
-		(pts
 			(xy 44.45 107.95) (xy 49.53 107.95)
 		)
@@
 	(wire
 		(pts
-			(xy 283.21 30.48) (xy 283.21 33.02)
-		)
-		(stroke
-			(width 0)
-			(type default)
-		)
-	)
-	(wire
-		(pts
 			(xy 73.66 36.83) (xy 82.55 36.83)
 		)
@@
 	)
 	(symbol
-		(lib_id "Device:R")
-		(at 314.96 46.99 90)
-		(unit 1)
-		(exclude_from_sim no)
-		(in_bom yes)
-		(on_board yes)
-		(dnp no)
-		(property "Reference" "R78"
-			(at 321.564 48.006 90)
-			(effects
-				(font
-					(size 1.27 1.27)
-				)
-				(justify left)
-			)
-		)
-		(property "Value" "150R"
-			(at 317.5 46.99 90)
-			(effects
-				(font
-					(size 1.27 1.27)
-				)
-				(justify left)
-			)
-		)
-		(property "Footprint" "Resistor_SMD:R_0603_1608Metric"
-			(at 314.96 48.768 90)
-			(effects
-				(font
-					(size 1.27 1.27)
-				)
-				(hide yes)
-			)
-		)
-		(property "Datasheet" "~"
-			(at 314.96 46.99 0)
-			(effects
-				(font
-					(size 1.27 1.27)
-				)
-				(hide yes)
-			)
-		)
-		(property "Description" "Resistor"
-			(at 314.96 46.99 0)
-			(effects
-				(font
-					(size 1.27 1.27)
-				)
-				(hide yes)
-			)
-		)
-		(property "JLC" "C22808"
-			(at 314.96 46.99 0)
-			(effects
-				(font
-					(size 1.27 1.27)
-				)
-				(hide yes)
-			)
-		)
-		(pin "1"
-		)
-		(pin "2"
-		)
-		(instances
-			(project "hw-openmower-universal"
-				(path "/e12e8a63-1d1b-4736-9aba-a87a258b2b11/2dcb05ea-788f-4ed6-923e-0b0051e68de3"
-					(reference "R78")
-					(unit 1)
-				)
-				(path "/e12e8a63-1d1b-4736-9aba-a87a258b2b11/35c1a146-5cd7-4cc8-a12d-17de73f02598"
-					(reference "R79")
-					(unit 1)
-				)
-				(path "/e12e8a63-1d1b-4736-9aba-a87a258b2b11/0359b790-c26c-4759-a59f-5a6b50a14036"
-					(reference "R80")
-					(unit 1)
-				)
-			)
-		)
-	)
-	(symbol
 		(lib_id "power:GND")
 		(at 267.97 45.72 270)
@@
 	(symbol
 		(lib_id "Device:R")
-		(at 283.21 26.67 0)
+		(at 130.81 139.7 90)
 		(unit 1)
 		(exclude_from_sim no)
@@
 		(dnp no)
 		(property "Reference" "R43"
-			(at 282.194 33.274 90)
+			(at 137.414 140.716 90)
 			(effects
 				(font
@@
 		)
 		(property "Value" "150R"
-			(at 283.21 29.21 90)
+			(at 133.35 139.7 90)
 			(effects
 				(font
@@
 		)
 		(property "Footprint" "Resistor_SMD:R_0603_1608Metric"
-			(at 281.432 26.67 90)
+			(at 130.81 141.478 90)
 			(effects
 				(font
@@
 		)
 		(property "Datasheet" "~"
-			(at 283.21 26.67 0)
+			(at 130.81 139.7 0)
 			(effects
 				(font
@@
 		)
 		(property "Description" "Resistor"
-			(at 283.21 26.67 0)
+			(at 130.81 139.7 0)
 			(effects
 				(font
@@
 		)
 		(property "JLC" "C22808"
-			(at 283.21 26.67 0)
+			(at 130.81 139.7 0)
 			(effects
 				(font

Commit message: wip
Connections:
- net GND: now also J36.5 (Pin_5); no longer J36.6 (Pin_6)
- net HALL_SENSOR.U: now also J36.2 (Pin_2); no longer J36.5 (Pin_5)
- net HALL_SENSOR.V: now also J36.4 (Pin_4); no longer J36.2 (Pin_2)
- net HALL_SENSOR.W: now also J36.6 (Pin_6); no longer J36.4 (Pin_4)
Changed lines of the file:
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@@
 	(wire
 		(pts
-			(xy 284.48 127) (xy 284.48 128.27)
+			(xy 271.78 127) (xy 271.78 128.27)
 		)
 		(stroke
@@
 	(wire
 		(pts
-			(xy 254 127) (xy 271.78 127)
+			(xy 306.07 127) (xy 284.48 127)
 		)
 		(stroke
@@
 	)
 	(label "HALL_SENSOR.U"
-		(at 254 127 0)
+		(at 306.07 121.92 180)
 		(fields_autoplaced yes)
 		(effects
@@
 				(size 1.27 1.27)
 			)
-			(justify left bottom)
+			(justify right bottom)
 		)
 	)
 	(label "HALL_SENSOR.V"
-		(at 306.07 121.92 180)
+		(at 306.07 124.46 180)
 		(fields_autoplaced yes)
 		(effects
@@
 	)
 	(label "HALL_SENSOR.W"
-		(at 306.07 124.46 180)
+		(at 306.07 127 180)
 		(fields_autoplaced yes)
 		(effects
@@
 	(symbol
 		(lib_id "power:GND")
-		(at 284.48 128.27 0)
+		(at 271.78 128.27 0)
+		(mirror y)
 		(unit 1)
 		(exclude_from_sim no)
@@
 		(fields_autoplaced yes)
 		(property "Reference" "#PWR085"
-			(at 284.48 134.62 0)
+			(at 271.78 134.62 0)
 			(effects
 				(font
@@
 		)
 		(property "Value" "GND"
-			(at 284.48 133.35 0)
+			(at 271.78 133.35 0)
 			(effects
 				(font
@@
 		)
 		(property "Footprint" ""
-			(at 284.48 128.27 0)
+			(at 271.78 128.27 0)
 			(effects
 				(font
@@
 		)
 		(property "Datasheet" ""
-			(at 284.48 128.27 0)
+			(at 271.78 128.27 0)
 			(effects
 				(font
@@
 		)
 		(property "Description" "Power symbol creates a global label with name \"GND\" , ground"
-			(at 284.48 128.27 0)
+			(at 271.78 128.27 0)
 			(effects
 				(font

Commit message: wip
Parts:
- removed C102, C105: 22uF/25V, Capacitor_SMD:C_0805_2012Metric, symbol Device:C
- removed C108: 10uF@50V, Capacitor_SMD:C_1206_3216Metric, symbol Device:C
- removed C111: 100nF@50V, Capacitor_SMD:C_0402_1005Metric, symbol Device:C
- removed D31: SS14, Diode_SMD:D_SMA, symbol Diode:SS14
- removed D4: VS-2EFH02HM3/I, Diode_SMD:D_SMF, symbol Device:D_Schottky
- removed R27, R28: R, Resistor_SMD:R_0201_0603Metric, symbol Device:R
- removed R31: 100k, Resistor_SMD:R_0402_1005Metric, symbol Device:R
- added C1: 10uF@50V, Capacitor_SMD:C_1206_3216Metric, symbol Device:C
- added C10, C3: 100nF@50V, Capacitor_SMD:C_0402_1005Metric, symbol Device:C
- added C35: 22uF/25V, Capacitor_SMD:C_0805_2012Metric, symbol Device:C
- added D22: VS-2EFH02HM3/I, Diode_SMD:D_SMF, symbol Device:D_Schottky
- added D4: SS14, Diode_SMD:D_SMA, symbol Diode:SS14
- added L5: 47uH, Inductor_SMD:L_Sunlord_SWPA5040S, symbol Device:L
- added R10: 120k, Resistor_SMD:R_0603_1608Metric, symbol Device:R
- added R17: 22k, Resistor_SMD:R_0603_1608Metric, symbol Device:R
- added R9: 100k, Resistor_SMD:R_0402_1005Metric, symbol Device:R
- C21: value 100nF@50V -> 22uF/25V; footprint Capacitor_SMD:C_0402_1005Metric -> Capacitor_SMD:C_0805_2012Metric; JLC C307331 -> C45783
Connections:
- net 5V: now also C21.1, C35.1, D4.1 (K), L5.2, R10.1; no longer U28.3 (FB)
- net 5V_Main: now also D4.2 (A)
- net GND: now also C21.2, C1.2, C3.2, C35.2, D22.2 (A), R17.2
- net VBATT: now also C1.1, C3.1, R9.1
- net at U28.1 (CB): now also C10.2; no longer C21.2
- net at U28.4 (~{SHDN}): now also R9.2
- net at U28.6 (SW): now also C10.1, D22.1 (K), L5.1; no longer C21.1
- new net: R10.2, R17.1, U28.3 (FB)

Commit message: wip
Parts:
- added D31, D36: LED GREEN, LED_SMD:LED_0805_2012Metric, symbol Device:LED
- added R45, R64: 1k, Resistor_SMD:R_0805_2012Metric, symbol Device:R
Connections:
- net 5V: now also D31.2 (A)
- net 5V_Main: now also D36.2 (A)
- net GND: now also R45.2, R64.2
- new net: D31.1 (K), R45.1
- new net: D36.1 (K), R64.1

Commit message: wip
Parts:
- added C76: 22pF/50V, Capacitor_SMD:C_0603_1608Metric, symbol Device:C
Connections:
- net GND: now also C76.2
- net SHUTDOWN: now also C76.1
Changed lines of the file:
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@@
 	)
 	(junction
+		(at 280.67 59.69)
+		(diameter 0)
+		(color 0 0 0 0)
+	)
+	(junction
 		(at 184.15 46.99)
 		(diameter 0)
@@
 	(wire
 		(pts
-			(xy 280.67 58.42) (xy 280.67 71.12)
+			(xy 280.67 58.42) (xy 280.67 59.69)
 		)
 		(stroke
@@
 	(wire
 		(pts
+			(xy 280.67 59.69) (xy 298.45 59.69)
+		)
+		(stroke
+			(width 0)
+			(type default)
+		)
+	)
+	(wire
+		(pts
 			(xy 191.77 124.46) (xy 243.84 124.46)
 		)
@@
 	(wire
 		(pts
+			(xy 280.67 59.69) (xy 280.67 71.12)
+		)
+		(stroke
+			(width 0)
+			(type default)
+		)
+	)
+	(wire
+		(pts
 			(xy 49.53 107.95) (xy 54.61 107.95)
 		)
@@
 	)
 	(symbol
+		(lib_id "Device:C")
+		(at 298.45 63.5 0)
+		(unit 1)
+		(exclude_from_sim no)
+		(in_bom yes)
+		(on_board yes)
+		(dnp no)
+		(fields_autoplaced yes)
+		(property "Reference" "C76"
+			(at 302.26 62.2299 0)
+			(effects
+				(font
+					(size 1.27 1.27)
+				)
+				(justify left)
+			)
+		)
+		(property "Value" "22pF/50V"
+			(at 302.26 64.7699 0)
+			(effects
+				(font
+					(size 1.27 1.27)
+				)
+				(justify left)
+			)
+		)
+		(property "Footprint" "Capacitor_SMD:C_0603_1608Metric"
+			(at 299.4152 67.31 0)
+			(effects
+				(font
+					(size 1.27 1.27)
+				)
+				(hide yes)
+			)
+		)
+		(property "Datasheet" "~"
+			(at 298.45 63.5 0)
+			(effects
+				(font
+					(size 1.27 1.27)
+				)
+				(hide yes)
+			)
+		)
+		(property "Description" "Unpolarized capacitor"
+			(at 298.45 63.5 0)
+			(effects
+				(font
+					(size 1.27 1.27)
+				)
+				(hide yes)
+			)
+		)
+		(property "JLC" "C1653"
+			(at 298.45 63.5 0)
+			(effects
+				(font
+					(size 1.27 1.27)
+				)
+				(hide yes)
+			)
+		)
+		(pin "1"
+		)
+		(pin "2"
+		)
+		(instances
+			(project "hw-openmower-universal"
+				(path "/e12e8a63-1d1b-4736-9aba-a87a258b2b11/2dcb05ea-788f-4ed6-923e-0b0051e68de3"
+					(reference "C76")
+					(unit 1)
+				)
+				(path "/e12e8a63-1d1b-4736-9aba-a87a258b2b11/35c1a146-5cd7-4cc8-a12d-17de73f02598"
+					(reference "C109")
+					(unit 1)
+				)
+				(path "/e12e8a63-1d1b-4736-9aba-a87a258b2b11/0359b790-c26c-4759-a59f-5a6b50a14036"
+					(reference "C110")
+					(unit 1)
+				)
+			)
+		)
+	)
+	(symbol
 		(lib_id "Device:D_TVS")
 		(at 218.44 113.03 180)
@@
 					(unit 1)
 				)
+			)
+		)
+	)
+	(symbol
+		(lib_id "power:GND")
+		(at 298.45 67.31 0)
+		(unit 1)
+		(exclude_from_sim no)
+		(in_bom yes)
+		(on_board yes)
+		(dnp no)
+		(fields_autoplaced yes)
+		(property "Reference" "#PWR0157"
+			(at 298.45 73.66 0)
+			(effects
+				(font
+					(size 1.27 1.27)
+				)
+				(hide yes)
+			)
+		)
+		(property "Value" "GND"
+			(at 298.45 72.39 0)
+			(effects
+				(font
+					(size 1.27 1.27)
+				)
+			)
+		)
+		(property "Footprint" ""
+			(at 298.45 67.31 0)
+			(effects
+				(font
+					(size 1.27 1.27)
+				)
+				(hide yes)
+			)
+		)
+		(property "Datasheet" ""
+			(at 298.45 67.31 0)
+			(effects
+				(font
+					(size 1.27 1.27)
+				)
+				(hide yes)
+			)
+		)
+		(property "Description" "Power symbol creates a global label with name \"GND\" , ground"
+			(at 298.45 67.31 0)
+			(effects
+				(font
+					(size 1.27 1.27)
+				)
+				(hide yes)
+			)
+		)
+		(pin "1"
+		)
+		(instances
+			(project "hw-openmower-universal"
+				(path "/e12e8a63-1d1b-4736-9aba-a87a258b2b11/2dcb05ea-788f-4ed6-923e-0b0051e68de3"
+					(reference "#PWR0157")
+					(unit 1)
+				)
+				(path "/e12e8a63-1d1b-4736-9aba-a87a258b2b11/35c1a146-5cd7-4cc8-a12d-17de73f02598"
+					(reference "#PWR0159")
+					(unit 1)
+				)
+				(path "/e12e8a63-1d1b-4736-9aba-a87a258b2b11/0359b790-c26c-4759-a59f-5a6b50a14036"
+					(reference "#PWR0160")
+					(unit 1)
+				)

Commit message: wip
Parts:
- D4: JLC (none) -> C2480
- J22: JLC (none) -> C557666
- J39: JLC (none) -> C557665
- J42: JLC (none) -> C428721
- J45: JLC (none) -> C7500843
- J48: now not fitted
- U28: JLC (none) -> C3200285
Connections:
- no-connect marks 9 -> 5

Commit message: First Version worth testing
Parts:
- J36: JLC (none) -> C5383104
Changed lines of the file:
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@@
+			)
+		)
+		(property "JLC" "C5383104"
+			(at 276.86 124.46 0)
+			(effects
+				(font
+					(size 1.27 1.27)
+				)
+				(hide yes)
 			)
 		)
