File: Connectors.kicad_sch (KiCad schematic)
At the start: 16 parts, among them J6 USB_A_Stacked, J7 HR911130A, J8 HR911130A, U3 TPS2065CDBV

Commit message: wip
Parts:
- removed C10: 100nF@50V, Capacitor_SMD:C_0402_1005Metric, symbol Device:C

Commit message: wip
Connections:
- net ETH1.PAIR_A_N: now also J7.3 (P3); no longer J7.2 (P2)
- net ETH1.PAIR_A_P: now also J7.2 (P2); no longer J7.3 (P3)
- net ETH1.PAIR_B_N: now also J7.7 (P7); no longer J7.4 (P4)
- net ETH1.PAIR_B_P: now also J7.4 (P4); no longer J7.7 (P7)
- net ETH1.PAIR_C_N: now also J7.6 (P6); no longer J7.5 (P5)
- net ETH1.PAIR_C_P: now also J7.5 (P5); no longer J7.6 (P6)
- net ETH1.PAIR_D_N: now also J7.9 (P9); no longer J7.8 (P8)
- net ETH1.PAIR_D_P: now also J7.8 (P8); no longer J7.9 (P9)
- net ETH2.PAIR_A_N: now also J8.3 (P3); no longer J8.2 (P2)
- net ETH2.PAIR_A_P: now also J8.2 (P2); no longer J8.3 (P3)
- net ETH2.PAIR_B_N: now also J8.7 (P7); no longer J8.4 (P4)
- net ETH2.PAIR_B_P: now also J8.4 (P4); no longer J8.7 (P7)
- net ETH2.PAIR_C_N: now also J8.6 (P6); no longer J8.5 (P5)
- net ETH2.PAIR_C_P: now also J8.5 (P5); no longer J8.6 (P6)
- net ETH2.PAIR_D_N: now also J8.9 (P9); no longer J8.8 (P8)
- net ETH2.PAIR_D_P: now also J8.8 (P8); no longer J8.9 (P9)
Changed lines of the file:
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@@
 	)
 	(label "ETH1.PAIR_D_P"
-		(at 205.74 132.08 0)
+		(at 205.74 129.54 0)
 		(fields_autoplaced yes)
 		(effects
@@
 	)
 	(label "ETH2.PAIR_C_P"
-		(at 205.74 212.09 0)
+		(at 205.74 209.55 0)
 		(fields_autoplaced yes)
 		(effects
@@
 	)
 	(label "ETH2.PAIR_B_P"
-		(at 205.74 214.63 0)
+		(at 205.74 207.01 0)
 		(fields_autoplaced yes)
 		(effects
@@
 	)
 	(label "ETH2.PAIR_D_N"
-		(at 205.74 217.17 0)
+		(at 205.74 219.71 0)
 		(fields_autoplaced yes)
 		(effects
@@
 	)
 	(label "ETH1.PAIR_A_N"
-		(at 205.74 114.3 0)
+		(at 205.74 116.84 0)
 		(fields_autoplaced yes)
 		(effects
@@
 	)
 	(label "ETH1.PAIR_D_N"
-		(at 205.74 129.54 0)
+		(at 205.74 132.08 0)
 		(fields_autoplaced yes)
 		(effects
@@
 	)
 	(label "ETH1.PAIR_A_P"
-		(at 205.74 116.84 0)
+		(at 205.74 114.3 0)
 		(fields_autoplaced yes)
 		(effects
@@
 	)
 	(label "ETH1.PAIR_B_N"
-		(at 205.74 119.38 0)
+		(at 205.74 127 0)
 		(fields_autoplaced yes)
 		(effects
@@
 	)
 	(label "ETH2.PAIR_D_P"
-		(at 205.74 219.71 0)
+		(at 205.74 217.17 0)
 		(fields_autoplaced yes)
 		(effects
@@
 	)
 	(label "ETH1.PAIR_C_N"
-		(at 205.74 121.92 0)
+		(at 205.74 124.46 0)
 		(fields_autoplaced yes)
 		(effects
@@
 	)
 	(label "ETH2.PAIR_C_N"
-		(at 205.74 209.55 0)
+		(at 205.74 212.09 0)
 		(fields_autoplaced yes)
 		(effects
@@
 	)
 	(label "ETH1.PAIR_C_P"
-		(at 205.74 124.46 0)
+		(at 205.74 121.92 0)
 		(fields_autoplaced yes)
 		(effects
@@
 	)
 	(label "ETH2.PAIR_B_N"
-		(at 205.74 207.01 0)
+		(at 205.74 214.63 0)
 		(fields_autoplaced yes)
 		(effects
@@
 	)
 	(label "ETH1.PAIR_B_P"
-		(at 205.74 127 0)
+		(at 205.74 119.38 0)
 		(fields_autoplaced yes)
 		(effects
@@
 	)
 	(label "ETH2.PAIR_A_N"
-		(at 205.74 201.93 0)
+		(at 205.74 204.47 0)
 		(fields_autoplaced yes)
 		(effects
@@
 	)
 	(label "ETH2.PAIR_A_P"
-		(at 205.74 204.47 0)
-		(fields_autoplaced yes)
-		(effects
+		(at 205.74 201.93 0)
+		(fields_autoplaced yes)
+		(effects

Commit message: wip
Connections:
- net ETH2.PAIR_D_N: now also J8.8 (P8); no longer J8.9 (P9)
- net ETH2.PAIR_D_P: now also J8.9 (P9); no longer J8.8 (P8)
Changed lines of the file:
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@@
 	)
 	(label "ETH2.PAIR_D_N"
-		(at 205.74 219.71 0)
+		(at 205.74 217.17 0)
 		(fields_autoplaced yes)
 		(effects
@@
 	)
 	(label "ETH2.PAIR_D_P"
-		(at 205.74 217.17 0)
+		(at 205.74 219.71 0)
 		(fields_autoplaced yes)
 		(effects
