File: hw-openmower-universal.kicad_sch (KiCad schematic)
At the start: 32 parts

Commit message: wip
Other:
- sheet subpcb_logic ports: added AGPIO[0..5]; removed AGPIO1, AGPIO2, AGPIO3, AGPIO4

Commit message: wip
Parts:
- added U1, U48, U49, U50, U51, U52: ~, mousebites:Mousebite_3, symbol mousebites:Mousebite_3
Connections:
- net AGPIO1: now also U49.3, U50.3
- net AGPIO2: now also U48.3, U51.3
- net AGPIO3: now also U1.3, U52.3
- net UART1.RX: now also U49.1, U50.1
- net UART1.TX: now also U49.2, U50.2
- net UART2.RX: now also U48.1, U51.1
- net UART2.TX: now also U48.2, U51.2
- net UART4.RX: now also U1.1, U52.1
- net UART4.TX: now also U1.2, U52.2

Commit message: wip
Parts:
- removed U50, U51, U52: ~, mousebites:Mousebite_3, symbol mousebites:Mousebite_3
- added U50: ~, mousebites:Mousebite_8, symbol mousebites:Mousebite_8
- U1, U48, U49: footprint mousebites:Mousebite_3 -> mousebites:Mousebite_4; symbol mousebites:Mousebite_3 -> mousebites:Mousebite_4
Connections:
- net 5V: now also U1.4, U48.4, U49.4, U50.5
- net AGPIO1: now also U50.8
- net GND: now also U50.3, U50.4
- net UART1.RX: now also U50.6
- net UART1.TX: now also U50.7
- net V_BATTERY: now also U50.1, U50.2

Commit message: wip
Parts:
- removed H11, H12, H16, H18, H19, H4, H8, H9: MountingHole_Pad, MountingHole:MountingHole_4.3mm_M4_Pad_Via, symbol Mechanical:MountingHole_Pad
- added U51, U52, U53: ~, mousebites:Mousebite_8, symbol mousebites:Mousebite_8
Connections:
- net 5V: now also U51.5, U52.5
- net AGPIO1: now also U50.6; no longer U50.8
- net AGPIO2: now also U51.6
- net AGPIO3: now also U52.6
- net GND: now also U51.3, U51.4, U52.3, U52.4, U53.5, U53.6, U53.7, U53.8
- net UART1.RX: now also U50.8; no longer U50.6
- net UART2.RX: now also U51.8
- net UART2.TX: now also U51.7
- net UART4.RX: now also U52.8
- net UART4.TX: now also U52.7
- net V_BATTERY: now also U51.1, U51.2, U52.1, U52.2, U53.1, U53.2, U53.3, U53.4
Other:
- removed sheet subpcb_aux
- sheet subpcb_logic ports: added none; removed GPIO14, RASPI_FAN_ON
- moved on the sheet: H10, H5, H6, H7

Commit message: wip
Parts:
- added U2, U4, U54, U55, U56, U57, U58, U59, U60: ~, mousebites:Mousebite_8, symbol mousebites:Mousebite_8
- added U61: ~, mousebites:Mousebite_4, symbol mousebites:Mousebite_4
Connections:
- net 5V: now also U1.3, U61.3; no longer U1.4, U48.4
- net AGPIO3: now also U60.7; no longer U1.3
- net GND: now also U1.4, U2.5, U2.6, U2.7, U2.8, U4.5, U4.6, U4.7, U4.8, U54.5, U54.6, U54.7, U54.8, U55.5, U55.6, U55.7, U55.8, U56.1, U56.2, U56.3, U56.4, U56.5, U56.6, U56.7, U56.8, U57.1, U57.2, U57.3, U57.4, U57.5, U57.6, U57.7, U57.8, U58.1, U58.2, U58.3, U58.4, U58.5, U58.6, U58.7, U58.8, U59.1, U59.2, U59.3, U59.4, U59.5, U59.6, U59.7, U59.8, U61.4
- net UART4.RX: now also U60.4; no longer U1.1
- net UART4.TX: now also U60.5; no longer U1.2
- net UART6.RX: now also U1.1, U60.2
- net UART6.TX: now also U1.2, U60.1
- net V_BATTERY: now also U2.1, U2.2, U2.3, U2.4, U4.1, U4.2, U4.3, U4.4, U54.1, U54.2, U54.3, U54.4, U55.1, U55.2, U55.3, U55.4
- new net I2C1.SCL: U48.4, U61.2
- new net I2C1.SDA: U60.8, U61.1
- no-connect marks 0 -> 2

Commit message: wip
Parts:
- added U62, U63, U64, U65, U66, U67, U68, U69, U70, U71: ~, mousebites:Mousebite_8, symbol mousebites:Mousebite_8
Connections:
- net AGPIO4: now also U60.1, U61.4
- net GND: now also U62.1, U62.2, U62.3, U62.4, U62.5, U62.6, U62.7, U62.8, U63.1, U63.2, U63.3, U63.4, U63.5, U63.6, U63.7, U63.8, U64.1, U64.2, U64.3, U64.4, U64.5, U64.6, U64.7, U64.8, U65.1, U65.2, U65.3, U65.4, U65.5, U65.6, U65.7, U65.8, U66.1, U66.2, U66.3, U66.4, U66.5, U66.6, U66.7, U66.8, U67.1, U67.2, U67.3, U67.4, U67.5, U67.6, U67.7, U67.8, U68.1, U68.2, U68.3, U68.4, U68.5, U68.6, U68.7, U68.8, U69.1, U69.2, U69.3, U69.4, U69.5, U69.6, U69.7, U69.8, U70.1, U70.2, U70.3, U70.4, U70.5, U70.6, U70.7, U70.8, U71.1, U71.2, U71.3, U71.4, U71.5, U71.6, U71.7, U71.8; no longer U61.4
- net UART6.RX: now also U60.3; no longer U60.2
- net UART6.TX: now also U60.2; no longer U60.1
- no-connect marks 2 -> 1
